File: schematic/controller.kicad_sch (KiCad schematic)
At the start: 38 parts, among them J5 Player 1, J6 Player 2, Q4 2N3904, Q5 2N3904, U18 74LS541, U19 74LS541, U24 74LS00

Commit message: fixed for github
Other:
- note added: "CTRL_EN_1 is Joypad ARM CRTL_EN_2 is Joypad FIRE"
Changed lines of the file:
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@@
     (stroke (width 0) (type default))
+  )
+  (text "CTRL_EN_1 is Joypad ARM\nCRTL_EN_2 is Joypad FIRE" (at 230.505 55.499 0)
+    (effects (font (size 1.27 1.27)) (justify left bottom))
   )
   (label "D7" (at 133.985 103.505 0) (fields_autoplaced)
